File: hardware/xrng2.sch (KiCad schematic (older format))
At the start: 27 parts

Commit message: IDs, footprints, DRC
Parts:
- added C115: 100u, Capacitors_SMD:C_0805_HandSoldering, symbol C
- added J102, J103: GS3, Connectors:GS3, symbol GS3
- added J104, J106: Conn_01x02, Pin_Headers:Pin_Header_Straight_1x02_Pitch2.54mm, symbol Conn_01x02
- added J105: Conn_01x03, Pin_Headers:Pin_Header_Straight_1x03_Pitch2.54mm, symbol Conn_01x03
- C101, C102, C103, C104, C105, C106, C107, C109, C110, C112, C113, C114: renamed from C?; footprint (none) -> Capacitors_SMD:C_0603_HandSoldering
- C108, C111: renamed from C?; value C -> 100n; footprint (none) -> Capacitors_SMD:C_0603_HandSoldering
- D101, D102: renamed from D?; footprint (none) -> Diodes_SMD:D_SOD-523
- J101: renamed from J?; footprint AVR-PDI-6 -> Pin_Headers:Pin_Header_Straight_2x03_Pitch2.54mm
- J107: renamed from J?; footprint (none) -> Connectors:USB_B
- R101, R102: renamed from R?; footprint (none) -> Resistors_SMD:R_0603_HandSoldering
- TP101, TP102: renamed from TP?; footprint (none) -> Measurement_Points:Measurement_Point_Square-SMD-Pad_Big
- U101: renamed from U?; footprint (none) -> Housings_SOIC:SOIC-14_3.9x8.7mm_Pitch1.27mm
- U102: renamed from U?; footprint TQFP64 -> Housings_QFP:TQFP-64_14x14mm_Pitch0.8mm
- U103: renamed from U?; footprint (none) -> Housings_SOIC:SOIC-14W_7.5x9.0mm_Pitch1.27mm
- Y101: renamed from Y?; footprint (none) -> kuro:SMD_Crystal_Multi_QC6CB_7A_ABM7
- gave numbers to parts that had none: 1
Connections:
- net +3V3: now also C115.1, J106.1 (Pin_1)
- net AVE_DIG: now also J103.2 (G2); no longer U102.21 (MOSI/XCK1/OC0CHS/OC1B/PC5)
- net GND: now also C115.2, J106.2 (Pin_2)
- net RO_OUT: now also J102.2 (G2); no longer U102.41 (PE5/OC1B/XCK1/MOSI)
- net at TP102.1: now also U102.8 (DAC0/AC2/ADC2/PB2); no longer U102.22 (MISO/RXD1/~OC0DLS~/PC6)
- net MULTIPLIER: now reaches U102.26 (OC0A/PD0)
- net at U102.27 (XCK0/OC0B/PD1): now also J105.1 (Pin_1)
- net at U102.28 (RXD0/OC0C/PD2): now also J105.2 (Pin_2)
- net at U102.29 (TXD0/OC0D/PD3): now also J105.3 (Pin_3)
- net at U102.30 (PD4/OC1A/~SS~): now also J104.1 (Pin_1)
- net at U102.31 (PD5/OC1B/XCK1/MOSI): now also J104.2 (Pin_2)
- net at U102.42 (PE6/RXD1/MISO/TOSC2): now also J102.3 (G3); no longer TP101.1
- net at U102.6 (AREFB/AC0/ADC0/PB0): now also TP101.1
- new net: J103.1 (G1), U102.21 (MOSI/XCK1/OC0CHS/OC1B/PC5)
- new net: J103.3 (G3), U102.22 (MISO/RXD1/~OC0DLS~/PC6)
- new net: J102.1 (G1), U102.41 (PE5/OC1B/XCK1/MOSI)
- no-connect marks 0 -> 27
Other:
- moved on the sheet: TP101, TP102

Commit message: Corrected ring oscillator wiring
Parts:
- U103: footprint Housings_SOIC:SOIC-14W_7.5x9.0mm_Pitch1.27mm -> Housings_SOIC:SOIC-14_3.9x8.7mm_Pitch1.27mm
Connections:
- net VA1: no longer U103.13 (1Dp), U103.3 (2A), U103.8 (1Dn)
- net VA2: no longer U103.1 (2Dp), U103.10 (3A), U103.5 (2Dn)
- new net VB1: U103.13 (1Dp), U103.3 (2A), U103.8 (1Dn)
- new net VB2: U103.1 (2Dp), U103.10 (3A), U103.5 (2Dn)
Changed lines of the file:
@@
 F 0 "U103" H 2100 4600 60  0000 C CNN
 F 1 "CD4007" H 2200 4500 60  0000 C CNN
-F 2 "Housings_SOIC:SOIC-14W_7.5x9.0mm_Pitch1.27mm" H 2450 3550 60  0001 C CNN
+F 2 "Housings_SOIC:SOIC-14_3.9x8.7mm_Pitch1.27mm" H 2450 3550 60  0001 C CNN
 F 3 "" H 2450 3550 60  0001 C CNN
 	1    3250 3950
@@
 	2900 4700 2900 4600
 Text Label 2900 4700 0    60   ~ 0
-VA1
+VB1
 Wire Wire Line
 	3550 4600 3550 4700
@@
 	3250 3250 3250 3300
 Text Label 3750 4700 0    60   ~ 0
-VA2
+VB2
 Text Label 2800 3200 0    60   ~ 0
-VA1
+VB1
 Wire Wire Line
 	2700 3300 2700 3200
@@
 	2700 3200 2800 3200
 Text Label 3550 3200 0    60   ~ 0
-VA2
+VB2
 Wire Wire Line
 	3450 3300 3450 3200
