File: hardware/xrng2.kicad_pcb (KiCad board)
At the start: 2 copper layers, 69 parts, among them J101 AVR-PDI-6A, J102 GS3, J103 GS3, J104 Conn_01x02, J105 Conn_01x03, J106 Conn_01x02, J107 USB_B, J301 GS2, Q301 MMBT3904, Q302 MMBT3904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

Commit message: Design rules for Seeed
Parts:
- moved U101 18.7 mm to (125.0, 25.0), turned to 90 degrees
- moved U103 5.08 mm to (125.0, 35.0), turned to 90 degrees
Connections:
- U103 pad 1: /VA2 -> /VB2
- U103 pad 10: /VA2 -> /VB2
- U103 pad 13: /VA1 -> /VB1
- U103 pad 3: /VA1 -> /VB1
- U103 pad 5: /VA2 -> /VB2
- U103 pad 8: /VA1 -> /VB1
Other:
- copper layers 2 -> 4
- rule trace_min: 0.2 -> 0.1524
- rule via_min_drill: 0.3 -> 0.2
- rule via_min_size: 0.4 -> 0.2
Changed lines of the file:
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@@
 (kicad_pcb (version 4) (host pcbnew 4.0.7)
   (general
-    (links 175)
-    (no_connects 175)
+    (links 173)
+    (no_connects 173)
     (area 0 0 0 0)
     (thickness 1.6)
@@
     (zones 0)
     (modules 69)
-    (nets 48)
+    (nets 50)
   )
   (page A4)
   (layers
     (0 F.Cu signal)
+    (1 PWR power)
+    (2 GND power)
     (31 B.Cu signal)
     (32 B.Adhes user)
@@
   (setup
     (last_trace_width 0.25)
+    (user_trace_width 0.1524)
+    (user_trace_width 0.2)
+    (user_trace_width 0.3)
+    (user_trace_width 0.5)
+    (user_trace_width 1)
     (trace_clearance 0.2)
     (zone_clearance 0.508)
     (zone_45_only no)
-    (trace_min 0.2)
+    (trace_min 0.1524)
     (segment_width 0.2)
     (edge_width 0.15)
     (via_size 0.6)
     (via_drill 0.4)
-    (via_min_size 0.4)
-    (via_min_drill 0.3)
+    (via_min_size 0.2)
+    (via_min_drill 0.2)
+    (user_via 0.4 0.2)
+    (user_via 0.5 0.3)
+    (user_via 0.6 0.4)
     (uvia_size 0.3)
     (uvia_drill 0.1)
@@
   (net 46 "Net-(U102-Pad38)")
   (net 47 "Net-(U102-Pad39)")
+  (net 48 /VB2)
+  (net 49 /VB1)
   (net_class Default "This is the default net class."
     (clearance 0.2)
@@
     (add_net /VA1)
     (add_net /VA2)
+    (add_net /VB1)
+    (add_net /VB2)
     (add_net AVE_ANA)
     (add_net AVE_DIG)
@@
   )
   (module Housings_SOIC:SOIC-14_3.9x8.7mm_Pitch1.27mm (layer F.Cu)
-    (at 138.3 38.19)
+    (at 125 25 90)
     (descr "14-Lead Plastic Small Outline (SL) - Narrow, 3.90 mm Body [SOIC] (see Microchip Packaging Specification 00000049BS.pdf)")
     (tags "SOIC 1.27")
     (attr smd)
-    (fp_text reference U101 (at 0 -5.375) (layer F.SilkS)
-      (effects (font (size 1 1) (thickness 0.15)))
-    )
-    (fp_text value CD4007 (at 0 5.375) (layer F.Fab)
-      (effects (font (size 1 1) (thickness 0.15)))
-    )
-    (fp_text user %R (at 0 0) (layer F.Fab)
+    (fp_text reference U101 (at 0 -5.375 90) (layer F.SilkS)
+      (effects (font (size 1 1) (thickness 0.15)))
+    )
+    (fp_text value CD4007 (at 0 5.375 90) (layer F.Fab)
+      (effects (font (size 1 1) (thickness 0.15)))
+    )
+    (fp_text user %R (at 0 0 90) (layer F.Fab)
       (effects (font (size 0.9 0.9) (thickness 0.135)))
     )
@@
     (fp_line (start -2.075 4.45) (end 2.075 4.45) (layer F.SilkS) (width 0.15))
     (fp_line (start -2.075 -4.425) (end -3.45 -4.425) (layer F.SilkS) (width 0.15))
-    (pad 1 smd rect (at -2.7 -3.81) (size 1.5 0.6) (layers F.Cu F.Paste F.Mask)
+    (pad 1 smd rect (at -2.7 -3.81 90) (size 1.5 0.6) (layers F.Cu F.Paste F.Mask)
       (net 42 /VA2))
-    (pad 2 smd rect (at -2.7 -2.54) (size 1.5 0.6) (layers F.Cu F.Paste F.Mask)
-      (net 1 +3V3))
-    (pad 3 smd rect (at -2.7 -1.27) (size 1.5 0.6) (layers F.Cu F.Paste F.Mask)
+    (pad 2 smd rect (at -2.7 -2.54 90) (size 1.5 0.6) (layers F.Cu F.Paste F.Mask)
+      (net 1 +3V3))
+    (pad 3 smd rect (at -2.7 -1.27 90) (size 1.5 0.6) (layers F.Cu F.Paste F.Mask)
       (net 43 /VA1))
-    (pad 4 smd rect (at -2.7 0) (size 1.5 0.6) (layers F.Cu F.Paste F.Mask)
-      (net 2 GND))
-    (pad 5 smd rect (at -2.7 1.27) (size 1.5 0.6) (layers F.Cu F.Paste F.Mask)
+    (pad 4 smd rect (at -2.7 0 90) (size 1.5 0.6) (layers F.Cu F.Paste F.Mask)
+      (net 2 GND))
+    (pad 5 smd rect (at -2.7 1.27 90) (size 1.5 0.6) (layers F.Cu F.Paste F.Mask)
       (net 42 /VA2))
-    (pad 6 smd rect (at -2.7 2.54) (size 1.5 0.6) (layers F.Cu F.Paste F.Mask)
+    (pad 6 smd rect (at -2.7 2.54 90) (size 1.5 0.6) (layers F.Cu F.Paste F.Mask)
       (net 3 /RO_OUT))
-    (pad 7 smd rect (at -2.7 3.81) (size 1.5 0.6) (layers F.Cu F.Paste F.Mask)
-      (net 2 GND))
-    (pad 8 smd rect (at 2.7 3.81) (size 1.5 0.6) (layers F.Cu F.Paste F.Mask)
+    (pad 7 smd rect (at -2.7 3.81 90) (size 1.5 0.6) (layers F.Cu F.Paste F.Mask)
+      (net 2 GND))
+    (pad 8 smd rect (at 2.7 3.81 90) (size 1.5 0.6) (layers F.Cu F.Paste F.Mask)
       (net 43 /VA1))
-    (pad 9 smd rect (at 2.7 2.54) (size 1.5 0.6) (layers F.Cu F.Paste F.Mask)
-      (net 2 GND))
-    (pad 10 smd rect (at 2.7 1.27) (size 1.5 0.6) (layers F.Cu F.Paste F.Mask)
+    (pad 9 smd rect (at 2.7 2.54 90) (size 1.5 0.6) (layers F.Cu F.Paste F.Mask)
+      (net 2 GND))
+    (pad 10 smd rect (at 2.7 1.27 90) (size 1.5 0.6) (layers F.Cu F.Paste F.Mask)
       (net 42 /VA2))
-    (pad 11 smd rect (at 2.7 0) (size 1.5 0.6) (layers F.Cu F.Paste F.Mask)
-      (net 1 +3V3))
-    (pad 12 smd rect (at 2.7 -1.27) (size 1.5 0.6) (layers F.Cu F.Paste F.Mask)
+    (pad 11 smd rect (at 2.7 0 90) (size 1.5 0.6) (layers F.Cu F.Paste F.Mask)
+      (net 1 +3V3))
+    (pad 12 smd rect (at 2.7 -1.27 90) (size 1.5 0.6) (layers F.Cu F.Paste F.Mask)
       (net 3 /RO_OUT))
-    (pad 13 smd rect (at 2.7 -2.54) (size 1.5 0.6) (layers F.Cu F.Paste F.Mask)
+    (pad 13 smd rect (at 2.7 -2.54 90) (size 1.5 0.6) (layers F.Cu F.Paste F.Mask)
       (net 43 /VA1))
-    (pad 14 smd rect (at 2.7 -3.81) (size 1.5 0.6) (layers F.Cu F.Paste F.Mask)
+    (pad 14 smd rect (at 2.7 -3.81 90) (size 1.5 0.6) (layers F.Cu F.Paste F.Mask)
       (net 1 +3V3))
     (model ${KISYS3DMOD}/Housings_SOIC.3dshapes/SOIC-14_3.9x8.7mm_Pitch1.27mm.wrl
@@
   )
   (module Housings_SOIC:SOIC-14_3.9x8.7mm_Pitch1.27mm (layer F.Cu)
-    (at 121.35 38.54)
+    (at 125 35 90)
     (descr "14-Lead Plastic Small Outline (SL) - Narrow, 3.90 mm Body [SOIC] (see Microchip Packaging Specification 00000049BS.pdf)")
     (tags "SOIC 1.27")
     (attr smd)
-    (fp_text reference U103 (at 0 -5.375) (layer F.SilkS)
-      (effects (font (size 1 1) (thickness 0.15)))
-    )
-    (fp_text value CD4007 (at 0 5.375) (layer F.Fab)
-      (effects (font (size 1 1) (thickness 0.15)))
-    )
-    (fp_text user %R (at 0 0) (layer F.Fab)
+    (fp_text reference U103 (at 0 -5.375 90) (layer F.SilkS)
+      (effects (font (size 1 1) (thickness 0.15)))
+    )
+    (fp_text value CD4007 (at 0 5.375 90) (layer F.Fab)
+      (effects (font (size 1 1) (thickness 0.15)))
+    )
+    (fp_text user %R (at 0 0 90) (layer F.Fab)
       (effects (font (size 0.9 0.9) (thickness 0.135)))
     )
@@
     (fp_line (start -2.075 4.45) (end 2.075 4.45) (layer F.SilkS) (width 0.15))
     (fp_line (start -2.075 -4.425) (end -3.45 -4.425) (layer F.SilkS) (width 0.15))
-    (pad 1 smd rect (at -2.7 -3.81) (size 1.5 0.6) (layers F.Cu F.Paste F.Mask)
-      (net 42 /VA2))
-    (pad 2 smd rect (at -2.7 -2.54) (size 1.5 0.6) (layers F.Cu F.Paste F.Mask)
-      (net 1 +3V3))
-    (pad 3 smd rect (at -2.7 -1.27) (size 1.5 0.6) (layers F.Cu F.Paste F.Mask)
-      (net 43 /VA1))
-    (pad 4 smd rect (at -2.7 0) (size 1.5 0.6) (layers F.Cu F.Paste F.Mask)
-      (net 2 GND))
-    (pad 5 smd rect (at -2.7 1.27) (size 1.5 0.6) (layers F.Cu F.Paste F.Mask)
-      (net 42 /VA2))
-    (pad 6 smd rect (at -2.7 2.54) (size 1.5 0.6) (layers F.Cu F.Paste F.Mask)
+    (pad 1 smd rect (at -2.7 -3.81 90) (size 1.5 0.6) (layers F.Cu F.Paste F.Mask)
+      (net 48 /VB2))
+    (pad 2 smd rect (at -2.7 -2.54 90) (size 1.5 0.6) (layers F.Cu F.Paste F.Mask)
+      (net 1 +3V3))
+    (pad 3 smd rect (at -2.7 -1.27 90) (size 1.5 0.6) (layers F.Cu F.Paste F.Mask)
+      (net 49 /VB1))
+    (pad 4 smd rect (at -2.7 0 90) (size 1.5 0.6) (layers F.Cu F.Paste F.Mask)
+      (net 2 GND))
+    (pad 5 smd rect (at -2.7 1.27 90) (size 1.5 0.6) (layers F.Cu F.Paste F.Mask)
+      (net 48 /VB2))
+    (pad 6 smd rect (at -2.7 2.54 90) (size 1.5 0.6) (layers F.Cu F.Paste F.Mask)
       (net 17 "Net-(D101-Pad1)"))
-    (pad 7 smd rect (at -2.7 3.81) (size 1.5 0.6) (layers F.Cu F.Paste F.Mask)
-      (net 2 GND))
-    (pad 8 smd rect (at 2.7 3.81) (size 1.5 0.6) (layers F.Cu F.Paste F.Mask)
-      (net 43 /VA1))
-    (pad 9 smd rect (at 2.7 2.54) (size 1.5 0.6) (layers F.Cu F.Paste F.Mask)
-      (net 2 GND))
-    (pad 10 smd rect (at 2.7 1.27) (size 1.5 0.6) (layers F.Cu F.Paste F.Mask)
-      (net 42 /VA2))
-    (pad 11 smd rect (at 2.7 0) (size 1.5 0.6) (layers F.Cu F.Paste F.Mask)
-      (net 1 +3V3))
-    (pad 12 smd rect (at 2.7 -1.27) (size 1.5 0.6) (layers F.Cu F.Paste F.Mask)
+    (pad 7 smd rect (at -2.7 3.81 90) (size 1.5 0.6) (layers F.Cu F.Paste F.Mask)
+      (net 2 GND))
+    (pad 8 smd rect (at 2.7 3.81 90) (size 1.5 0.6) (layers F.Cu F.Paste F.Mask)
+      (net 49 /VB1))
+    (pad 9 smd rect (at 2.7 2.54 90) (size 1.5 0.6) (layers F.Cu F.Paste F.Mask)
+      (net 2 GND))
+    (pad 10 smd rect (at 2.7 1.27 90) (size 1.5 0.6) (layers F.Cu F.Paste F.Mask)
+      (net 48 /VB2))
+    (pad 11 smd rect (at 2.7 0 90) (size 1.5 0.6) (layers F.Cu F.Paste F.Mask)
+      (net 1 +3V3))
+    (pad 12 smd rect (at 2.7 -1.27 90) (size 1.5 0.6) (layers F.Cu F.Paste F.Mask)
       (net 17 "Net-(D101-Pad1)"))
-    (pad 13 smd rect (at 2.7 -2.54) (size 1.5 0.6) (layers F.Cu F.Paste F.Mask)
-      (net 43 /VA1))
-    (pad 14 smd rect (at 2.7 -3.81) (size 1.5 0.6) (layers F.Cu F.Paste F.Mask)
+    (pad 13 smd rect (at 2.7 -2.54 90) (size 1.5 0.6) (layers F.Cu F.Paste F.Mask)
+      (net 49 /VB1))
+    (pad 14 smd rect (at 2.7 -3.81 90) (size 1.5 0.6) (layers F.Cu F.Paste F.Mask)
       (net 1 +3V3))
     (model ${KISYS3DMOD}/Housings_SOIC.3dshapes/SOIC-14_3.9x8.7mm_Pitch1.27mm.wrl

Commit message: Sub circuit layouts
Parts:
- moved C108 123.0 mm to (119.2, 21.5), turned to 90 degrees
- moved J103 121.4 mm to (78.5, 95.7)
- moved C111 117.2 mm to (119.2, 31.5), turned to 90 degrees
- moved R307 110.2 mm to (197.5, 33.2)
- moved C302 108.2 mm to (193.0, 36.2), turned to 180 degrees
- moved R304 104.4 mm to (192.0, 33.2)
- moved C107 103.6 mm to (131.8, 26.8), turned to 270 degrees
- moved R101 102.5 mm to (133.8, 26.8), turned to 270 degrees
- moved R102 97.2 mm to (133.8, 35.8), turned to 270 degrees
- moved R204 86.0 mm to (202.2, 70.2)
- moved R303 85.4 mm to (185.0, 42.2), turned to 90 degrees
- moved R308 83.0 mm to (186.8, 36.2)
- moved C301 82.8 mm to (180.5, 36.5), turned to 180 degrees
- moved R302 82.0 mm to (171.8, 39.2)
- moved C304 81.5 mm to (187.5, 47.5), turned to 90 degrees
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Routing:
- net AVE_ANA: track 0.00 -> 23.6 mm, vias 0 -> 2
- net Net-(C304-Pad1): track 0.00 -> 21.7 mm
- net /VB1: track 0.00 -> 15.2 mm
- net /VA1: track 0.00 -> 15.2 mm
- net Net-(R304-Pad2): track 0.00 -> 15.2 mm
- net /VB2: track 0.00 -> 12.0 mm, vias 0 -> 3
- net /VA2: track 0.00 -> 12.0 mm, vias 0 -> 3
- net Net-(C303-Pad1): track 0.00 -> 11.4 mm
- net Net-(C303-Pad2): track 0.00 -> 9.22 mm
- net Net-(R303-Pad2): track 0.00 -> 8.84 mm
- net Net-(C305-Pad1): track 0.00 -> 8.52 mm
- net /RO_OUT: track 0.00 -> 8.15 mm
- net Net-(D101-Pad1): track 0.00 -> 8.00 mm
- net Net-(R304-Pad1): track 0.00 -> 7.93 mm
- net +3V3: track 0.00 -> 6.44 mm
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
Commit message: Dimensions and layout
Parts:
- C203: footprint Capacitors_SMD:C_0603_HandSoldering -> Capacitors_SMD:C_0805_HandSoldering
- moved J107 202.3 mm to (54.0, 111.8), turned to 180 degrees
- moved C112 189.9 mm to (60.2, 117.2)
- moved U104 185.8 mm to (59.2, 113.2), turned to 270 degrees
- moved C113 177.8 mm to (63.2, 111.0), turned to 270 degrees
- moved C114 172.0 mm to (66.0, 111.0), turned to 270 degrees
- moved C115 166.0 mm to (69.0, 111.0), turned to 270 degrees
- moved R307 154.1 mm to (58.4, 99.7), turned to 270 degrees
- moved U302 150.3 mm to (50.2, 93.4), turned to 270 degrees
- moved C302 149.7 mm to (55.4, 95.2), turned to 90 degrees
- moved C304 149.4 mm to (44.2, 89.7), turned to 0 degrees
- moved R304 146.8 mm to (58.4, 94.2), turned to 270 degrees
- moved C305 144.7 mm to (42.9, 85.2), turned to 90 degrees
- moved R306 143.1 mm to (45.2, 85.2), turned to 270 degrees
- moved R303 142.8 mm to (49.4, 87.2), turned to 0 degrees
- moved R308 141.5 mm to (55.4, 88.9), turned to 270 degrees
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Routing:
- net GND: track 0.00 -> 80.0 mm, vias 0 -> 42
- net +3V3: track 6.44 -> 82.3 mm, vias 0 -> 22
- net VBUS: track 0.00 -> 69.3 mm
- net /USB_DP: track 0.00 -> 45.2 mm
- net /USB_DM: track 0.00 -> 43.9 mm
- net AVE_DIG: track 0.00 -> 33.1 mm
- net /PDI_CLK: track 0.00 -> 28.7 mm, vias 0 -> 1
- net Net-(J105-Pad1): track 0.00 -> 28.0 mm, vias 0 -> 1
- net AVE_ANA: track 23.6 -> 49.8 mm, vias 2 -> 4
- net MULTIPLIER: track 0.00 -> 25.7 mm, vias 0 -> 2
- net Net-(J105-Pad2): track 0.00 -> 23.4 mm, vias 0 -> 1
- net Net-(J105-Pad3): track 0.00 -> 22.7 mm, vias 0 -> 1
- net Net-(J104-Pad1): track 0.00 -> 22.0 mm, vias 0 -> 1
- net Net-(J104-Pad2): track 0.00 -> 21.3 mm, vias 0 -> 1
- net /PDI_DAT: track 0.00 -> 19.9 mm, vias 0 -> 1
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- added copper zone on PWR, net +3V3
- added copper zone on GND, net GND
Other:
- board outline added: 70 x 60 mm

Commit message: Tracking finished
Routing:
- net VPP: track 17.3 -> 122.6 mm
- net /RO_OUT: track 20.0 -> 33.3 mm
- net +3V3: track 82.3 -> 82.9 mm
Changed lines of the file:
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@@
     (thickness 1.6)
     (drawings 6)
-    (tracks 512)
+    (tracks 533)
     (zones 0)
     (modules 69)
@@
     (arrow2b (pts (xy 39.936939 137.131669) (xy 41.063443 136.545248)))
   )
+  (segment (start 79.37 98.16) (end 79.41 98.16) (width 0.5) (layer F.Cu) (net 1))
+  (segment (start 79.41 98.16) (end 80.75 99.5) (width 0.5) (layer F.Cu) (net 1))
+  (via (at 80.75 99.5) (size 0.6) (drill 0.4) (layers F.Cu B.Cu) (net 1))
   (segment (start 69 109.75) (end 68.75 109.75) (width 1) (layer F.Cu) (net 1))
   (segment (start 68.75 109.75) (end 67.75 108.75) (width 1) (layer F.Cu) (net 1))
@@
   (segment (start 68.47 76.16) (end 67.17 76.16) (width 0.5) (layer F.Cu) (net 1))
   (via (at 67.17 76.16) (size 0.6) (drill 0.4) (layers F.Cu B.Cu) (net 1))
-  (segment (start 79.37 98.16) (end 80.67 98.16) (width 0.5) (layer F.Cu) (net 1))
-  (via (at 80.67 98.16) (size 0.6) (drill 0.4) (layers F.Cu B.Cu) (net 1))
   (segment (start 66.92 93.36) (end 66.92 94.66) (width 0.5) (layer F.Cu) (net 1))
   (via (at 66.92 94.66) (size 0.6) (drill 0.4) (layers F.Cu B.Cu) (net 1))
@@
   (segment (start 55.42 72.81) (end 55.42 71.16) (width 0.5) (layer F.Cu) (net 2))
   (via (at 55.42 71.16) (size 0.6) (drill 0.4) (layers F.Cu B.Cu) (net 2))
+  (segment (start 93.5 81) (end 95.62 78.88) (width 0.5) (layer F.Cu) (net 3))
+  (segment (start 95.62 78.88) (end 95.62 77.16) (width 0.5) (layer F.Cu) (net 3))
+  (segment (start 93.5 87.465) (end 93.5 81) (width 0.5) (layer F.Cu) (net 3))
+  (segment (start 91.67 88.16) (end 92.805 88.16) (width 0.5) (layer F.Cu) (net 3))
+  (segment (start 92.805 88.16) (end 93.5 87.465) (width 0.5) (layer F.Cu) (net 3))
   (segment (start 95.62 77.16) (end 95.62 75.16) (width 0.25) (layer F.Cu) (net 3))
   (segment (start 98.32 77.16) (end 95.62 77.16) (width 0.25) (layer F.Cu) (net 3))
@@
   (segment (start 95.92 99.56) (end 98.92 99.56) (width 0.5) (layer F.Cu) (net 7))
   (segment (start 98.92 99.56) (end 101.37 99.56) (width 0.5) (layer F.Cu) (net 7))
+  (segment (start 107 91.5) (end 107 87.39) (width 0.5) (layer F.Cu) (net 8))
+  (segment (start 107 87.39) (end 106.37 86.76) (width 0.5) (layer F.Cu) (net 8))
+  (segment (start 105.75 92.75) (end 107 91.5) (width 0.5) (layer F.Cu) (net 8))
+  (segment (start 95 92.75) (end 105.75 92.75) (width 0.5) (layer F.Cu) (net 8))
+  (segment (start 94.42 93.33) (end 95 92.75) (width 0.5) (layer F.Cu) (net 8))
+  (segment (start 94.42 97.91) (end 94.42 93.33) (width 0.5) (layer F.Cu) (net 8))
+  (segment (start 106.42 78.41) (end 106.42 84.11) (width 0.5) (layer F.Cu) (net 8))
+  (segment (start 106.42 84.11) (end 106.37 84.16) (width 0.5) (layer F.Cu) (net 8))
+  (segment (start 53.17 66.81) (end 53.17 65.71) (width 0.5) (layer F.Cu) (net 8))
+  (segment (start 53.17 65.71) (end 57.88 61) (width 0.5) (layer F.Cu) (net 8))
+  (segment (start 57.88 61) (end 107.5 61) (width 0.5) (layer F.Cu) (net 8))
+  (segment (start 107.5 61) (end 108.5 62) (width 0.5) (layer F.Cu) (net 8))
+  (segment (start 108.5 62) (end 108.5 77.25) (width 0.5) (layer F.Cu) (net 8))
+  (segment (start 108.5 77.25) (end 107.34 78.41) (width 0.5) (layer F.Cu) (net 8))
+  (segment (start 107.34 78.41) (end 106.42 78.41) (width 0.5) (layer F.Cu) (net 8))
   (segment (start 96.42 97.06) (end 99.07 97.06) (width 0.5) (layer F.Cu) (net 8))
   (segment (start 99.07 97.06) (end 99.47 96.66) (width 0.5) (layer F.Cu) (net 8))
