File: hardware/xrng2.kicad_pcb (KiCad board)
At the start: 4 copper layers, 70 x 60 mm, 69 parts, among them J101 AVR-PDI-6A, J102 GS3, J103 GS3, J104 Conn_01x02, J105 Conn_01x03, J106 Conn_01x02, J107 USB_B, J301 GS2, Q301 MMBT3904, Q302 MMBT3904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

Commit message: DRC OK
Routing:
- net +3V3: track 82.9 -> 84.9 mm
- net GND: track 80.0 -> 81.3 mm
Changed lines of the file:
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@@
   (general
     (links 173)
-    (no_connects 138)
-    (area 0 0 0 0)
+    (no_connects 0)
+    (area 38.524999 59.924999 134.85 139.83167)
     (thickness 1.6)
     (drawings 6)
-    (tracks 533)
+    (tracks 536)
     (zones 0)
     (modules 69)
@@
     (pad_to_mask_clearance 0.2)
     (aux_axis_origin 0 0)
-    (visible_elements FFFFFF7F)
+    (visible_elements 7FFFFFFF)
     (pcbplotparams
       (layerselection 0x00030_80000001)
@@
     (arrow2b (pts (xy 39.936939 137.131669) (xy 41.063443 136.545248)))
   )
+  (segment (start 103.87 64.6) (end 103.87 62.67) (width 0.5) (layer F.Cu) (net 1))
+  (segment (start 103.87 62.67) (end 103.7 62.5) (width 0.5) (layer F.Cu) (net 1))
   (segment (start 79.37 98.16) (end 79.41 98.16) (width 0.5) (layer F.Cu) (net 1))
   (segment (start 79.41 98.16) (end 80.75 99.5) (width 0.5) (layer F.Cu) (net 1))
@@
   (segment (start 105.36 64.6) (end 105.42 64.66) (width 0.5) (layer F.Cu) (net 1))
   (via (at 105.42 64.66) (size 0.6) (drill 0.4) (layers F.Cu B.Cu) (net 1))
-  (segment (start 103.72 64.45) (end 103.87 64.6) (width 0.5) (layer F.Cu) (net 1))
   (segment (start 55.42 96.11) (end 55.42 97.66) (width 0.5) (layer F.Cu) (net 1))
   (via (at 55.42 97.66) (size 0.6) (drill 0.4) (layers F.Cu B.Cu) (net 1))
@@
   (segment (start 55.17 83.61) (end 52.075 83.61) (width 0.5) (layer F.Cu) (net 1))
   (segment (start 52.075 96.11) (end 55.42 96.11) (width 0.5) (layer F.Cu) (net 1))
+  (segment (start 101.8 62.5) (end 101.8 63.7) (width 0.5) (layer F.Cu) (net 2))
+  (segment (start 101.8 63.7) (end 101.75 63.75) (width 0.5) (layer F.Cu) (net 2))
+  (via (at 101.75 63.75) (size 0.6) (drill 0.4) (layers F.Cu B.Cu) (net 2))
   (segment (start 42.92 84.21) (end 42.92 82.83) (width 0.5) (layer F.Cu) (net 2))
   (segment (start 42.92 82.83) (end 43 82.75) (width 0.5) (layer F.Cu) (net 2))
@@
   (segment (start 48.265 89.005) (end 48.17 88.91) (width 0.5) (layer F.Cu) (net 2))
   (via (at 48.17 88.91) (size 0.6) (drill 0.4) (layers F.Cu B.Cu) (net 2))
-  (via (at 48.5 76) (size 0.6) (drill 0.4) (layers F.Cu B.Cu) (net 2))
   (segment (start 55.17 81.71) (end 55.17 80.16) (width 0.5) (layer F.Cu) (net 2))
   (via (at 55.17 80.16) (size 0.6) (drill 0.4) (layers F.Cu B.Cu) (net 2))
@@
   (segment (start 49.82 75.01) (end 49.67 74.86) (width 0.5) (layer F.Cu) (net 13))
   (segment (start 55.42 75.01) (end 52.42 75.01) (width 0.5) (layer F.Cu) (net 13))
+  (segment (start 41.5 88.165) (end 41.5 82.25) (width 0.5) (layer F.Cu) (net 14))
+  (segment (start 41.5 82.25) (end 43.5 80.25) (width 0.5) (layer F.Cu) (net 14))
+  (segment (start 43.22 89.66) (end 42.995 89.66) (width 0.5) (layer F.Cu) (net 14))
+  (segment (start 42.995 89.66) (end 41.5 88.165) (width 0.5) (layer F.Cu) (net 14))
   (segment (start 45.17 80.27) (end 43.52 80.27) (width 0.5) (layer F.Cu) (net 14))
   (segment (start 43.52 80.27) (end 43.5 80.25) (width 0.5) (layer F.Cu) (net 14))
   (via (at 43.5 80.25) (size 0.6) (drill 0.4) (layers F.Cu B.Cu) (net 14))
-  (segment (start 47.25 75.25) (end 48.89 73.61) (width 0.5) (layer F.Cu) (net 14))
-  (segment (start 47.25 82.55) (end 47.25 75.25) (width 0.5) (layer F.Cu) (net 14))
-  (segment (start 48.8 83) (end 47.7 83) (width 0.5) (layer F.Cu) (net 14))
-  (segment (start 47.7 83) (end 47.25 82.55) (width 0.5) (layer F.Cu) (net 14))
   (segment (start 50.805 78.21) (end 50.805 79.485) (width 0.5) (layer F.Cu) (net 14))
   (segment (start 50.805 79.485) (end 50.02 80.27) (width 0.5) (layer F.Cu) (net 14))
@@
   (segment (start 78.12 78.13) (end 78.25 78) (width 0.5) (layer F.Cu) (net 19))
   (via (at 78.25 78) (size 0.6) (drill 0.4) (layers F.Cu B.Cu) (net 19))
-  (segment (start 77.145 78) (end 76.149998 78) (width 0.5) (layer B.Cu) (net 20))
-  (segment (start 76.149998 78) (end 72.399998 74.25) (width 0.5) (layer B.Cu) (net 20))
-  (segment (start 72.399998 74.25) (end 61.25 74.25) (width 0.5) (layer B.Cu) (net 20))
+  (segment (start 77.15 78.3) (end 76.449998 78.3) (width 0.5) (layer B.Cu) (net 20))
+  (segment (start 76.449998 78.3) (end 72.399998 74.25) (width 0.5) (layer B.Cu) (net 20))
   (segment (start 61.25 74.25) (end 59.5 72.5) (width 0.5) (layer B.Cu) (net 20))
-  (segment (start 60.25 67.467919) (end 60.507919 67.21) (width 0.5) (layer B.Cu) (net 20))
-  (segment (start 59.5 72.5) (end 59.5 68.25) (width 0.5) (layer B.Cu) (net 20))
   (segment (start 59.5 68.25) (end 60.25 67.5) (width 0.5) (layer B.Cu) (net 20))
+  (segment (start 72.399998 74.25) (end 61.25 74.25) (width 0.5) (layer B.Cu) (net 20))
+  (segment (start 59.5 72.5) (end 59.5 68.25) (width 0.5) (layer B.Cu) (net 20))
   (segment (start 60.25 67.5) (end 60.25 67.467919) (width 0.5) (layer B.Cu) (net 20))
+  (segment (start 60.25 67.467919) (end 60.507919 67.21) (width 0.5) (layer B.Cu) (net 20))
   (segment (start 60.507919 67.21) (end 61.71 67.21) (width 0.5) (layer B.Cu) (net 20))
-  (segment (start 77.32 79.76) (end 77.32 78.175) (width 0.5) (layer F.Cu) (net 20))
-  (segment (start 77.32 78.175) (end 77.145 78) (width 0.5) (layer F.Cu) (net 20))
-  (via (at 77.145 78) (size 0.6) (drill 0.4) (layers F.Cu B.Cu) (net 20))
+  (segment (start 77.32 79.76) (end 77.32 78.47) (width 0.5) (layer F.Cu) (net 20))
+  (segment (start 77.32 78.47) (end 77.15 78.3) (width 0.5) (layer F.Cu) (net 20))
+  (via (at 77.15 78.3) (size 0.6) (drill 0.4) (layers F.Cu B.Cu) (net 20))
   (segment (start 85.42 87.06) (end 86.455002 87.06) (width 0.5) (layer F.Cu) (net 21))
   (segment (start 86.455002 87.06) (end 88.825002 89.43) (width 0.5) (layer F.Cu) (net 21))
@@
   (segment (start 53.75 106) (end 52 107.75) (width 0.5) (layer F.Cu) (net 32))
   (segment (start 52 107.75) (end 52 109.25) (width 0.5) (layer F.Cu) (net 32))
+  (segment (start 45.17 84.06) (end 45.17 81.55) (width 0.5) (layer F.Cu) (net 33))
   (segment (start 70.02 91.06) (end 71.57 91.06) (width 0.5) (layer F.Cu) (net 33))
   (segment (start 71.57 91.06) (end 71.92 91.41) (width 0.5) (layer F.Cu) (net 33))
@@
   (segment (start 45.17 84.06) (end 47.815 84.06) (width 0.5) (layer F.Cu) (net 33))
   (segment (start 47.815 84.06) (end 48.265 83.61) (width 0.5) (layer F.Cu) (net 33))
-  (segment (start 45.17 81.55) (end 45.17 84.06) (width 0.5) (layer F.Cu) (net 33))
   (segment (start 47.72 65.16) (end 47.72 67.91) (width 0.5) (layer F.Cu) (net 34))
   (segment (start 47.72 67.91) (end 47.67 67.96) (width 0.5) (layer F.Cu) (net 34))

Commit message: F.Fab clean-up
Other:
- board text added: "1"
- board text added: "PDI"
- board text added: "Y101"
