File: hardware/xrng2.kicad_pcb (KiCad board)
At the start: 4 copper layers, 70 x 60 mm, 69 parts, among them J101 AVR-PDI-6A, J102 GS3, J103 GS3, J104 Conn_01x02, J105 Conn_01x03, J106 Conn_01x02, J107 USB_B, J301 GS2, Q301 MMBT3904, Q302 MMBT3904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

Commit message: I2C on expansion
Parts:
- added R103: 2k2, Resistors_SMD:R_0603_HandSoldering, B.Cu at (84.2, 101.8)
- added R104: 2k2, Resistors_SMD:R_0603_HandSoldering, B.Cu at (89.2, 101.8)
Connections:
- U102 pad 30: Net-(J104-Pad1) -> (no net)
- U102 pad 31: Net-(J104-Pad2) -> (no net)
- U102 pad 36: (no net) -> Net-(J104-Pad1)
- U102 pad 37: (no net) -> Net-(J104-Pad2)
Routing:
- net Net-(J104-Pad2): track 21.3 -> 31.7 mm
- net Net-(J104-Pad1): track 22.0 -> 28.8 mm
- net +3V3: track 84.9 -> 88.4 mm, vias 22 -> 24
Other:
- board text added: "C103"
- board text added: "C112"
- board text added: "C113"
- board text added: "C114"
- board text added: "C115"
- board text added: "C301"
- board text added: "C302"
- board text added: "C303"
- board text added: "C304"
- board text added: "C305"
- board text added: "J107"
- board text added: "J301"
- board text added: "Q301"
- board text added: "Q302"
- board text added: "R301"
- board text added: "R302"
- board text added: "R303"
- board text added: "R304"
- board text added: "R305"
- board text added: "R306"
- board text added: "R307"
- board text added: "RX"
- board text added: "TX"
- board text added: "U104"
- board text added: "U301"
- board text added: "U302"
- board text added: "XCK"
- board text removed: "1"
- board text removed: "PDI"
- board text removed: "Y101"

Commit message: Silk labels
Other:
- board text added: "1"
- board text added: "3V3"
- board text added: "ADC2"
- board text added: "AREFB"
- board text added: "C101"
- board text added: "C102"
- board text added: "C104"
- board text added: "C105"
- board text added: "C106"
- board text added: "C107"
- board text added: "C108"
- board text added: "C109"
- board text added: "C110"
- board text added: "C111"
- board text added: "C201"
- board text added: "C202"
- board text added: "C203"
- board text added: "C204"
- board text added: "C205"
- board text added: "C206"
- board text added: "C207"
- board text added: "D101"
- board text added: "D102"
- board text added: "D201"
- board text added: "D202"
- board text added: "D203"
- board text added: "D204"
- board text added: "GND"
- board text added: "J101"
- board text added: "J103"
- board text added: "L201"
- board text added: "MISO"
- board text added: "MOSI"
- board text added: "PDI"
- board text added: "R101"
- board text added: "R102"
- board text added: "R103"
- board text added: "R104"
- board text added: "R201"
- board text added: "R202"
- board text added: "R203"
- board text added: "R204"
- board text added: "R308"
- board text added: "SCL"
- board text added: "SDA"
- board text added: "U101"
- board text added: "U102"
- board text added: "U103"
- board text added: "U201"
- board text added: "VPP"
- board text added: "Y101"
Changed lines of the file:
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@@
     (area 39.924999 59.924999 110.075001 120.075001)
     (thickness 1.6)
-    (drawings 34)
+    (drawings 84)
     (tracks 548)
     (zones 0)
@@
     (47 F.CrtYd user)
     (48 B.Fab user)
-    (49 F.Fab user)
+    (49 F.Fab user hide)
   )
   (setup
-    (last_trace_width 0.25)
+    (last_trace_width 0.1524)
     (user_trace_width 0.1524)
     (user_trace_width 0.2)
@@
     )
   )
-  (gr_text TX (at 80.5 114) (layer Eco1.User)
-    (effects (font (size 1 1) (thickness 0.15)))
-  )
-  (gr_text TX (at 78 114) (layer Eco1.User)
-    (effects (font (size 1 1) (thickness 0.15)))
-  )
-  (gr_text RX (at 75.5 114) (layer Eco1.User)
-    (effects (font (size 1 1) (thickness 0.15)))
-  )
-  (gr_text XCK (at 72.75 114) (layer Eco1.User)
-    (effects (font (size 1 1) (thickness 0.15)))
-  )
-  (gr_text C114 (at 66 115.5) (layer Eco1.User)
-    (effects (font (size 1 1) (thickness 0.15)))
-  )
-  (gr_text C113 (at 63.25 107) (layer Eco1.User)
-    (effects (font (size 1 1) (thickness 0.15)))
-  )
+  (gr_text R308 (at 57 88.75 90) (layer Eco1.User)
+    (effects (font (size 1 1) (thickness 0.15)))
+  )
+  (gr_text Y101 (at 76.25 71.25 90) (layer Eco1.User)
+    (effects (font (size 1 1) (thickness 0.15)))
+  )
+  (gr_text C106 (at 89.75 84.25 90) (layer Eco1.User)
+    (effects (font (size 1 1) (thickness 0.15)))
+  )
+  (gr_text C101 (at 89.75 92.25 90) (layer Eco1.User)
+    (effects (font (size 1 1) (thickness 0.15)))
+  )
+  (gr_text MISO (at 75 101.5 90) (layer Eco1.User)
+    (effects (font (size 1 1) (thickness 0.15)))
+  )
+  (gr_text MOSI (at 72.25 101.5 90) (layer Eco1.User)
+    (effects (font (size 1 1) (thickness 0.15)))
+  )
+  (gr_text C102 (at 78.25 99.75) (layer Eco1.User)
+    (effects (font (size 1 1) (thickness 0.15)))
+  )
+  (gr_text J103 (at 69.5 98.5) (layer Eco1.User)
+    (effects (font (size 1 1) (thickness 0.15)))
+  )
+  (gr_text R102 (at 90.5 78.75) (layer Eco1.User)
+    (effects (font (size 1 1) (thickness 0.15)))
+  )
+  (gr_text R103 (at 84.25 100.25) (layer Eco2.User)
+    (effects (font (size 1 1) (thickness 0.15)) (justify mirror))
+  )
+  (gr_text R104 (at 89.25 100.25 360) (layer Eco2.User)
+    (effects (font (size 1 1) (thickness 0.15)) (justify mirror))
+  )
+  (gr_text ADC2 (at 62.75 84.5) (layer Eco1.User)
+    (effects (font (size 1 1) (thickness 0.15)))
+  )
+  (gr_text AREFB (at 62.75 78.25) (layer Eco1.User)
+    (effects (font (size 1 1) (thickness 0.15)))
+  )
+  (gr_text U102 (at 68 80.75 90) (layer Eco1.User)
+    (effects (font (size 1 1) (thickness 0.15)))
+  )
+  (gr_text 1 (at 69.25 67.25) (layer Eco1.User)
+    (effects (font (size 1 1) (thickness 0.15)))
+  )
+  (gr_text PDI (at 67 64.5) (layer Eco1.User)
+    (effects (font (size 1 1) (thickness 0.15)))
+  )
+  (gr_text J101 (at 61.75 64.5) (layer Eco1.User)
+    (effects (font (size 1 1) (thickness 0.15)))
+  )
+  (gr_text C104 (at 69.5 74.75) (layer Eco1.User)
+    (effects (font (size 1 1) (thickness 0.15)))
+  )
+  (gr_text C110 (at 73.25 70.25) (layer Eco1.User)
+    (effects (font (size 1 1) (thickness 0.15)))
+  )
+  (gr_text C109 (at 79.25 70.25) (layer Eco1.User)
+    (effects (font (size 1 1) (thickness 0.15)))
+  )
+  (gr_text C105 (at 83.25 74.75) (layer Eco1.User)
+    (effects (font (size 1 1) (thickness 0.15)))
+  )
+  (gr_text U103 (at 89 63) (layer Eco1.User)
+    (effects (font (size 1 1) (thickness 0.15)))
+  )
+  (gr_text U101 (at 99 63) (layer Eco1.User)
+    (effects (font (size 1 1) (thickness 0.15)))
+  )
+  (gr_text C111 (at 94.75 61.25) (layer Eco1.User)
+    (effects (font (size 1 1) (thickness 0.15)))
+  )
+  (gr_text C108 (at 102.75 61.25) (layer Eco1.User)
+    (effects (font (size 1 1) (thickness 0.15)))
+  )
+  (gr_text D101 (at 95 73.75) (layer Eco1.User)
+    (effects (font (size 1 1) (thickness 0.15)))
+  )
+  (gr_text C107 (at 99.5 73.75) (layer Eco1.User)
+    (effects (font (size 1 1) (thickness 0.15)))
+  )
+  (gr_text D102 (at 95 78.75) (layer Eco1.User)
+    (effects (font (size 1 1) (thickness 0.15)))
+  )
+  (gr_text R101 (at 99.5 78.75) (layer Eco1.User)
+    (effects (font (size 1 1) (thickness 0.15)))
+  )
+  (gr_text VPP (at 106.25 75.75) (layer Eco1.User)
+    (effects (font (size 1 1) (thickness 0.15)))
+  )
+  (gr_text D203 (at 101.75 87.75) (layer Eco1.User)
+    (effects (font (size 1 1) (thickness 0.15)))
+  )
+  (gr_text D202 (at 106 82.75) (layer Eco1.User)
+    (effects (font (size 1 1) (thickness 0.15)))
+  )
+  (gr_text C204 (at 101.75 82.75) (layer Eco1.User)
+    (effects (font (size 1 1) (thickness 0.15)))
+  )
+  (gr_text R204 (at 96.75 82.75) (layer Eco1.User)
+    (effects (font (size 1 1) (thickness 0.15)))
+  )
+  (gr_text C206 (at 107 88.75 90) (layer Eco1.User)
+    (effects (font (size 1 1) (thickness 0.15)))
+  )
+  (gr_text C207 (at 101 90.25 90) (layer Eco1.User)
+    (effects (font (size 1 1) (thickness 0.15)))
+  )
+  (gr_text C205 (at 96.5 87 90) (layer Eco1.User)
+    (effects (font (size 1 1) (thickness 0.15)))
+  )
+  (gr_text D204 (at 96.5 91 90) (layer Eco1.User)
+    (effects (font (size 1 1) (thickness 0.15)))
+  )
+  (gr_text D201 (at 94.25 95.75 90) (layer Eco1.User)
+    (effects (font (size 1 1) (thickness 0.15)))
+  )
+  (gr_text L201 (at 107.75 98 90) (layer Eco1.User)
+    (effects (font (size 1 1) (thickness 0.15)))
+  )
+  (gr_text U201 (at 103.75 96.75 90) (layer Eco1.User)
+    (effects (font (size 1 1) (thickness 0.15)))
+  )
+  (gr_text C202 (at 100.5 95.25) (layer Eco1.User)
+    (effects (font (size 1 1) (thickness 0.15)))
+  )
+  (gr_text R203 (at 97.5 100.75 90) (layer Eco1.User)
+    (effects (font (size 1 1) (thickness 0.15)))
+  )
+  (gr_text R202 (at 94.25 100.75 90) (layer Eco1.User)
+    (effects (font (size 1 1) (thickness 0.15)))
+  )
+  (gr_text C201 (at 107.5 103.5 90) (layer Eco1.User)
+    (effects (font (size 1 1) (thickness 0.15)))
+  )
+  (gr_text R201 (at 102.5 106.25) (layer Eco1.User)
+    (effects (font (size 1 1) (thickness 0.15)))
+  )
+  (gr_text C203 (at 97.5 106.25) (layer Eco1.User)
+    (effects (font (size 1 1) (thickness 0.15)))
+  )
+  (gr_text 3V3 (at 88 113 90) (layer Eco1.User)
+    (effects (font (size 1 1) (thickness 0.15)))
+  )
+  (gr_text GND (at 85.5 113 90) (layer Eco1.User)
+    (effects (font (size 1 1) (thickness 0.15)))
+  )
+  (gr_text SCL (at 83 113 90) (layer Eco1.User)
+    (effects (font (size 1 1) (thickness 0.15)))
+  )
+  (gr_text SDA (at 80.5 113 90) (layer Eco1.User)
+    (effects (font (size 1 1) (thickness 0.15)))
+  )
+  (gr_text TX (at 78 113.5 90) (layer Eco1.User)
+    (effects (font (size 1 1) (thickness 0.15)))
+  )
+  (gr_text RX (at 75.5 113.5 90) (layer Eco1.User)
+    (effects (font (size 1 1) (thickness 0.15)))
+  )
+  (gr_text XCK (at 73 113 90) (layer Eco1.User)
+    (effects (font (size 1 1) (thickness 0.15)))
+  )
+  (gr_text C114 (at 66 115) (layer Eco1.User)
+    (effects (font (size 1 1) (thickness 0.15)))
+  )
+  (gr_text C113 (at 63.25 108.25) (layer Eco1.User)
+    (effects (font (size 1 1) (thickness 0.15)))
+  )

Commit message: Silkscreen outlines
Other:
- board text added: "???"
