File: hardware/BoostSupply.sch (KiCad schematic (older format))
At the start: 9 parts

Commit message: IDs, footprints, DRC
Parts:
- added C204, C205, C206, C207: 1u, Capacitors_SMD:C_0603_HandSoldering, symbol C
- added D202, D203, D204: D, Diodes_SMD:D_SOD-523, symbol D
- added R204: 240, Resistors_SMD:R_0603_HandSoldering, symbol R
- added TP201: TEST, Measurement_Points:Measurement_Point_Square-SMD-Pad_Big, symbol TEST
- C201, C202, C203: renamed from C?; footprint (none) -> Capacitors_SMD:C_0603_HandSoldering
- L201: renamed from L?; footprint Inductors_NEOSID:Neosid_Inductor_SM-NE29_SMD1008 -> Resistors_SMD:R_0805_HandSoldering
- R201, R202, R203: renamed from R?; footprint (none) -> Resistors_SMD:R_0603_HandSoldering
- U201: renamed from U?; footprint (none) -> TO_SOT_Packages_SMD:SOT-23-5
- gave numbers to parts that had none: 1
Connections:
- net GND: now also C206.2, C207.2, D204.2 (A)
- net VPP: now also C206.1, D202.1 (K), TP201.1
- new net: C204.1, C205.1, R204.2
- new net: C205.2, D203.2 (A), D204.1 (K)
- new net: C204.2, C207.1, D202.2 (A), D203.1 (K)
- new net MULTIPLIER: R204.1

Commit message: Changed cap to 0805
Parts:
- C203: footprint Capacitors_SMD:C_0603_HandSoldering -> Capacitors_SMD:C_0805_HandSoldering
Changed lines of the file:
@@
 F 0 "C203" H 4700 3600 50  0000 L CNN
 F 1 "4.7u" H 4700 3500 50  0000 L CNN
-F 2 "Capacitors_SMD:C_0603_HandSoldering" H 4638 3400 50  0001 C CNN
+F 2 "Capacitors_SMD:C_0805_HandSoldering" H 4638 3400 50  0001 C CNN
 F 3 "" H 4600 3550 50  0001 C CNN
 	1    4600 3550

Commit message: 16V output parts
Parts:
- D201: BOM_PartNo MBR1020VL -> SS13FL/SD103BW
- L201: BOM_PartNo 74479887310 -> LQM21FN100M80L
- R202: value 130k -> 162k
- R203: value 13.3k -> 14k
Other:
- note added: "16V"
Changed lines of the file:
@@
 F 2 "Resistors_SMD:R_0805_HandSoldering" H 3250 2500 50  0001 C CNN
 F 3 "" H 3250 2500 50  0001 C CNN
-F 4 "74479887310" V 3350 2500 50  0000 C CNN "BOM_PartNo"
+F 4 "LQM21FN100M80L" V 3350 2500 50  0000 C CNN "BOM_PartNo"
 	1    3250 2500
 	0    1    -1   0
@@
 F 2 "Diodes_SMD:D_SOD-123F" H 4250 2500 50  0001 C CNN
 F 3 "" H 4250 2500 50  0001 C CNN
-F 4 "MBR1020VL" H 4250 2600 50  0000 C CNN "BOM_PartNo"
+F 4 "SS13FL/SD103BW" H 4250 2600 50  0000 C CNN "BOM_PartNo"
 	1    4250 2500
 	-1   0    0    -1
@@
 P 3900 3550
 F 0 "R203" H 3950 3600 50  0000 L CNN
-F 1 "13.3k" H 3950 3500 50  0000 L CNN
+F 1 "14k" H 3950 3500 50  0000 L CNN
 F 2 "Resistors_SMD:R_0603_HandSoldering" V 3830 3550 50  0001 C CNN
 F 3 "" H 3900 3550 50  0001 C CNN
@@
 P 4250 2900
 F 0 "R202" V 4450 2900 50  0000 C CNN
-F 1 "130k" V 4350 2900 50  0000 C CNN
+F 1 "162k" V 4350 2900 50  0000 C CNN
 F 2 "Resistors_SMD:R_0603_HandSoldering" V 4180 2900 50  0001 C CNN
 F 3 "" H 4250 2900 50  0001 C CNN
@@
 	5750 5000 5750 4950
 Connection ~ 5400 5000
+Text Notes 4900 2500 0    60   ~ 0
+16V
 $EndSCHEMATC
